File: LittleBenv2.kicad_sch (KiCad schematic)
At the start: 49 parts, among them J1 Conn_01x10, J2 Conn_01x10, J3 Conn_01x08, J4 Conn_02x05_Odd_Even, J5 Conn_01x08, J6 Oled, J7 Conn_01x02, Q1 2N3906, Q2 2N3906, SW1 Rotary_Encoder_Switch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

Commit message: Panel Update
Parts:
- C2: value CP -> 22uf
Changed lines of the file:
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@@
       (effects (font (size 1.27 1.27)) (justify left))
     )
-    (property "Value" "CP" (id 1) (at 326.8472 36.703 0)
+    (property "Value" "22uf" (id 1) (at 326.8472 36.703 0)
       (effects (font (size 1.27 1.27)) (justify left))
     )
@@
     )
     (path "/00000000-0000-0000-0000-000060977c40"
-      (reference "C2") (unit 1) (value "CP") (footprint "Capacitor_THT:CP_Radial_D6.3mm_P2.50mm")
+      (reference "C2") (unit 1) (value "22uf") (footprint "Capacitor_THT:CP_Radial_D6.3mm_P2.50mm")
     )
     (path "/00000000-0000-0000-0000-000060979af9"
